File: Keithley_17X_USB.kicad_pcb (KiCad board)
At the start: 2 copper layers, 70.5 x 44 mm, 42 parts, among them J1 USB_B, J2 SIGNAL INPUT, J3 PROG, U1 TLP281-4, U2 TLP281-4, U3 MIC5504-3.3YM5, U4 MSP430FR2110, U5 FT230XS

Commit message: Update Keithley_17X_USB.kicad_pcb
Parts:
- moved J3 70.5 mm to (112.3, 52.4), turned to 270 degrees
- moved D8 53.7 mm to (69.2, 108.9), turned to 90 degrees
- moved R7 51.9 mm to (71.7, 109.5), turned to 90 degrees
- moved C1 3.34 mm to (117.4, 60.5)
- moved C2 3.34 mm to (117.4, 66.8)
- moved U3 3.34 mm to (117.4, 63.7)
- moved C3 0.65 mm to (94.3, 71.2)
- moved C4 0.65 mm to (96.3, 71.2)
- turned H2 to 180 degrees
- turned H3 to 180 degrees
Connections:
- U4 pad 10: /CLK -> /SIGN
- U4 pad 7: /OVERRANGE -> /CLK
- U4 pad 8: /SIGN -> /D5
- U4 pad 9: /D5 -> /OVERRANGE
Routing:
- net /OVERRANGE: track 0.00 -> 17.6 mm
- net /SIGN: track 0.00 -> 16.8 mm
- net +3V3: track 2.28 -> 17.4 mm
- net /B2: track 0.00 -> 10.0 mm
- net +5V: track 27.4 -> 17.4 mm
- net /D5: track 0.00 -> 9.58 mm
- net /B1: track 0.00 -> 9.22 mm
- net /CLK: track 0.00 -> 8.80 mm
- net GND: track 25.9 -> 30.9 mm, vias 19 -> 23
- net /RXLED: track 1.56 -> 0.00 mm, vias 1 -> 0
Other:
- board text added: "3V3"
- board text added: "GND"
- board text added: "TCK"
- board text added: "TDIO"

Commit message: Update Keithley_17X_USB.kicad_pcb
Parts:
- moved JP1 54.5 mm to (111.1, 90.1), turned to 270 degrees
- moved R9 52.8 mm to (102.2, 90.1), turned to 180 degrees
- moved R8 52.1 mm to (114.9, 90.1), turned to 180 degrees
- moved R5 13.1 mm to (121.5, 72.2)
- moved D6 13.1 mm to (125.2, 72.2)
- moved C2 6.91 mm to (110.5, 67.1), turned to 90 degrees
- moved C1 5.09 mm to (113.7, 64.0)
- moved U3 5.09 mm to (113.7, 67.1)
- moved D5 4.35 mm to (125.2, 58.2)
- moved R4 4.35 mm to (121.5, 58.2)
- moved D4 3.85 mm to (125.2, 61.3)
- moved R3 3.85 mm to (121.5, 61.3)
- moved D1 3.85 mm to (128.7, 64.8)
- moved D3 3.85 mm to (120.5, 66.2)
- moved TH1 3.85 mm to (125.2, 66.2)
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Routing:
- net /B8: track 0.00 -> 14.0 mm, vias 0 -> 1
- net /RXLED: track 0.00 -> 13.6 mm, vias 0 -> 2
- net +3V3: track 17.4 -> 30.8 mm
- net /VCCIO: track 11.8 -> 23.7 mm
- net /TXLED: track 0.00 -> 11.0 mm
- net /B4: track 0.00 -> 10.9 mm
- net /RXD: track 0.00 -> 5.24 mm, vias 0 -> 2
- net /TXD: track 0.00 -> 3.47 mm
- net /SBWTDIO: track 0.11 -> 2.52 mm
- net Net-(D6-Pad2): track 0.02 -> 1.98 mm
- net +5V: track 17.4 -> 18.0 mm
- added copper zone on F.Cu, net +3V3
- added copper zone on F.Cu, net +5V
