File: Keithley_17X_USB.kicad_pcb (KiCad board)
At the start: 2 copper layers, 70.5 x 44 mm, 42 parts, among them J1 USB_B, J2 SIGNAL INPUT, J3 PROG, U1 TLP281-4, U2 TLP281-4, U3 MIC5504-3.3YM5, U4 MSP430FR2110, U5 FT230XS

Commit message: draft layout, need to cleanup and make pretty
Parts:
- moved R7 54.9 mm to (110.5, 70.7), turned to 270 degrees
- moved D8 53.8 mm to (110.5, 74.3)
- moved C3 10.9 mm to (104.3, 67.2), turned to 90 degrees
- moved C4 7.31 mm to (102.3, 67.2), turned to 90 degrees
- moved R8 6.39 mm to (109.8, 86.2), turned to 270 degrees
- moved R9 6.35 mm to (107.2, 86.2), turned to 90 degrees
- moved U4 1.41 mm to (103.3, 72.2)
Routing:
- net /SBWTDIO: track 2.52 -> 35.9 mm
- net /SBWTCK: track 0.04 -> 28.9 mm
- net /RATE: track 0.00 -> 21.7 mm, vias 0 -> 2
- net +3V3: track 30.8 -> 48.5 mm, vias 0 -> 2
- net /B8: track 14.0 -> 29.2 mm, vias 1 -> 4
- net /B4: track 10.9 -> 25.1 mm, vias 0 -> 4
- net /RXD: track 5.24 -> 16.0 mm
- net /TXD: track 3.47 -> 13.5 mm
- net /READ: track 0.00 -> 7.08 mm
- net /B2: track 10.0 -> 13.9 mm, vias 0 -> 2
- net Net-(JP1-Pad1): track 0.00 -> 3.59 mm
- net Net-(JP1-Pad3): track 0.00 -> 3.58 mm
- net /B1: track 9.22 -> 12.6 mm, vias 0 -> 2
- net Net-(D7-Pad2): track 0.00 -> 2.00 mm
- net Net-(D8-Pad2): track 0.00 -> 1.97 mm
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- added copper zone on F.Cu, net GND

Commit message: Update Keithley_17X_USB.kicad_pcb
Parts:
- moved R8 4.81 mm to (109.8, 81.4)
- moved R9 4.81 mm to (107.2, 81.4)
- moved JP1 4.81 mm to (111.1, 85.3)
- moved J3 3.00 mm to (112.3, 55.4)
Routing:
- net +3V3: track 48.5 -> 41.9 mm
- net /RATE: track 21.7 -> 16.9 mm
- net /SBWTDIO: track 35.9 -> 32.1 mm
- net /SBWTCK: track 28.9 -> 25.8 mm
- net /TXD: track 13.5 -> 11.7 mm
- net /RXD: track 16.0 -> 14.8 mm
Other:
- board text added: "CLK"
- board text added: "D5"

Commit message: Update Keithley_17X_USB.kicad_pcb
Parts:
- moved J3 2.85 mm to (112.3, 58.2)
- moved R8 0.96 mm to (109.8, 82.4)
- moved R9 0.96 mm to (107.2, 82.4)
- moved JP1 0.96 mm to (111.1, 86.2)
- moved D1 0.80 mm to (128.7, 65.5)
- moved H1 0.30 mm to (95.6, 52.7)
- moved H4 0.30 mm to (121.5, 52.7)
- moved H2 0.30 mm to (95.6, 89.8)
- moved H3 0.30 mm to (121.5, 89.8)
- moved U1 0.25 mm to (88.0, 78.8)
- moved J2 0.12 mm to (78.0, 63.6)
Routing:
- net +3V3: track 41.9 -> 52.5 mm
- net Net-(D1-Pad1): track 0.00 -> 8.95 mm
- net +5V: track 18.0 -> 25.6 mm
- net /B8: track 29.2 -> 24.8 mm, vias 4 -> 2
- net /B4: track 25.1 -> 22.2 mm, vias 4 -> 2
- net /SBWTDIO: track 32.1 -> 30.1 mm
- net Net-(D3-Pad2): track 0.00 -> 1.75 mm
- net /RATE: track 16.9 -> 17.8 mm
- net /B1_IN: track 11.5 -> 12.4 mm
- net /B2_IN: track 11.8 -> 12.6 mm
- net /B8_IN: track 10.8 -> 11.7 mm
- removed copper zone on F.Cu, net +3V3
- removed copper zone on F.Cu, net +5V
- removed copper zone on F.Cu, net GND
- removed copper zone on F.Cu, net Net-(D1-Pad1)
- removed copper zone on F.Cu, net Net-(D3-Pad2)
Other:
- outline, holes or cut-outs redrawn
