File: pcb/Keithley_17X_USB.sch (KiCad schematic (older format))
At the start: 42 parts, among them J1 USB_B, J2 SIGNAL INPUT, J3 PROG, U1 TLP281-4, U2 TLP281-4, U3 MIC5504-3.3YM5, U4 MSP430FR2110, U5 FT230XS

Commit message: add LEDs part number
Parts:
- D4, D5, D6, D7, D8: Description (none) -> Red 615~630nm 0805 Light Emitting Diodes (LED) RoHS; Manufacture (none) -> Foshan NationStar Optoelectronics; Mfg Part Number (none) -> NCD0805R1; Supplier (none) -> LCSC; Supplier Part Number (none) -> C84256
Changed lines of the file:
@@
 F 1 "RXLED" H 9550 6000 50  0000 C CNN
 F 2 "LED_SMD:LED_0805_2012Metric" H 9550 6100 50  0001 C CNN
-F 3 "~" H 9550 6100 50  0001 C CNN
+F 3 "https://datasheet.lcsc.com/szlcsc/1912191206_Foshan-NationStar-Optoelectronics-NCD0805R1_C84256.pdf" H 9550 6100 50  0001 C CNN
+F 4 "Red 615~630nm 0805 Light Emitting Diodes (LED) RoHS" H 9550 6100 50  0001 C CNN "Description"
+F 5 "Foshan NationStar Optoelectronics" H 9550 6100 50  0001 C CNN "Manufacture"
+F 6 "NCD0805R1" H 9550 6100 50  0001 C CNN "Mfg Part Number"
+F 7 "LCSC" H 9550 6100 50  0001 C CNN "Supplier"
+F 8 "C84256" H 9550 6100 50  0001 C CNN "Supplier Part Number"
 	1    9550 6100
 	0    -1   -1   0
@@
 F 1 "TXLED" H 9850 6000 50  0000 C CNN
 F 2 "LED_SMD:LED_0805_2012Metric" H 9850 6100 50  0001 C CNN
-F 3 "~" H 9850 6100 50  0001 C CNN
+F 3 "https://datasheet.lcsc.com/szlcsc/1912191206_Foshan-NationStar-Optoelectronics-NCD0805R1_C84256.pdf" H 9850 6100 50  0001 C CNN
+F 4 "Red 615~630nm 0805 Light Emitting Diodes (LED) RoHS" H 9850 6100 50  0001 C CNN "Description"
+F 5 "Foshan NationStar Optoelectronics" H 9850 6100 50  0001 C CNN "Manufacture"
+F 6 "NCD0805R1" H 9850 6100 50  0001 C CNN "Mfg Part Number"
+F 7 "LCSC" H 9850 6100 50  0001 C CNN "Supplier"
+F 8 "C84256" H 9850 6100 50  0001 C CNN "Supplier Part Number"
 	1    9850 6100
 	0    -1   -1   0
@@
 F 1 "READ" H 10250 6000 50  0000 C CNN
 F 2 "LED_SMD:LED_0805_2012Metric" H 10250 6100 50  0001 C CNN
-F 3 "~" H 10250 6100 50  0001 C CNN
+F 3 "https://datasheet.lcsc.com/szlcsc/1912191206_Foshan-NationStar-Optoelectronics-NCD0805R1_C84256.pdf" H 10250 6100 50  0001 C CNN
+F 4 "Red 615~630nm 0805 Light Emitting Diodes (LED) RoHS" H 10250 6100 50  0001 C CNN "Description"
+F 5 "Foshan NationStar Optoelectronics" H 10250 6100 50  0001 C CNN "Manufacture"
+F 6 "NCD0805R1" H 10250 6100 50  0001 C CNN "Mfg Part Number"
+F 7 "LCSC" H 10250 6100 50  0001 C CNN "Supplier"
+F 8 "C84256" H 10250 6100 50  0001 C CNN "Supplier Part Number"
 	1    10250 6100
 	0    -1   -1   0
@@
 F 1 "5V" H 8800 6000 50  0000 C CNN
 F 2 "LED_SMD:LED_0805_2012Metric" H 8800 6100 50  0001 C CNN
-F 3 "~" H 8800 6100 50  0001 C CNN
+F 3 "https://datasheet.lcsc.com/szlcsc/1912191206_Foshan-NationStar-Optoelectronics-NCD0805R1_C84256.pdf" H 8800 6100 50  0001 C CNN
+F 4 "Red 615~630nm 0805 Light Emitting Diodes (LED) RoHS" H 8800 6100 50  0001 C CNN "Description"
+F 5 "Foshan NationStar Optoelectronics" H 8800 6100 50  0001 C CNN "Manufacture"
+F 6 "NCD0805R1" H 8800 6100 50  0001 C CNN "Mfg Part Number"
+F 7 "LCSC" H 8800 6100 50  0001 C CNN "Supplier"
+F 8 "C84256" H 8800 6100 50  0001 C CNN "Supplier Part Number"
 	1    8800 6100
 	0    -1   -1   0
@@
 F 1 "3V3" H 9100 6000 50  0000 C CNN
 F 2 "LED_SMD:LED_0805_2012Metric" H 9100 6100 50  0001 C CNN
-F 3 "~" H 9100 6100 50  0001 C CNN
+F 3 "https://datasheet.lcsc.com/szlcsc/1912191206_Foshan-NationStar-Optoelectronics-NCD0805R1_C84256.pdf" H 9100 6100 50  0001 C CNN
+F 4 "Red 615~630nm 0805 Light Emitting Diodes (LED) RoHS" H 9100 6100 50  0001 C CNN "Description"
+F 5 "Foshan NationStar Optoelectronics" H 9100 6100 50  0001 C CNN "Manufacture"
+F 6 "NCD0805R1" H 9100 6100 50  0001 C CNN "Mfg Part Number"
+F 7 "LCSC" H 9100 6100 50  0001 C CNN "Supplier"
+F 8 "C84256" H 9100 6100 50  0001 C CNN "Supplier Part Number"
 	1    9100 6100
 	0    -1   -1   0
